File: pcb-pico-i2c.kicad/pcb-pico-i2c.kicad_sch (KiCad schematic)
At the start: 7 parts, among them J1 Grove, J2 Connector_Pico_I2C, J3 Stemma QT, J4 RUN, J5 3V3_EN, SW1 SW_Push, SW2 SW_Push

Commit message: changes for Rev3 of board
Parts:
- added J6: 3V3, user:PinHole_1x01, symbol Connector_Generic:Conn_01x01
- added JP1, JP2: SolderJumper_2_Bridged, Jumper:SolderJumper-2_P1.3mm_Bridged_Pad1.0x1.5mm, symbol Jumper:SolderJumper_2_Bridged
- added R1, R2: R, Resistor_SMD:R_0402_1005Metric, symbol Device:R
Connections:
- net at J1.3, J2.1 (3V3), J3.2 (Vcc): now also J6.1 (Pin_1), JP1.1 (A), JP2.1 (A)
- net at J1.1, J2.5 (SCL), J3.4 (SCL): now also R1.2
- net at J1.2, J2.6 (SDA), J3.3 (SDA): now also R2.2
- new net: JP1.2 (B), R1.1
- new net: JP2.2 (B), R2.1
Changed lines of the file:
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@@
   (title_block
     (title "Pico I2C-Connector (no-solder)")
-    (date "2022-06-27")
-    (rev "2")
+    (date "2022-07-18")
+    (rev "3")
     (company "Bernhard Bablok")
     (comment 1 "https://github.com/bablokb/pcb-pico-i2c")
@@
   (junction (at 116.205 94.615) (diameter 0) (color 0 0 0 0)
   )
+  (junction (at 106.68 98.425) (diameter 0) (color 0 0 0 0)
+  )
   (junction (at 102.87 104.775) (diameter 0) (color 0 0 0 0)
   )
+  (junction (at 102.87 90.17) (diameter 0) (color 0 0 0 0)
+  )
   (junction (at 111.125 102.235) (diameter 0) (color 0 0 0 0)
   )
   (junction (at 107.95 77.47) (diameter 0) (color 0 0 0 0)
   )
+  (junction (at 54.61 94.615) (diameter 0) (color 0 0 0 0)
+  )
   (junction (at 106.68 107.315) (diameter 0) (color 0 0 0 0)
   )
@@
     (stroke (width 0) (type default) (color 0 0 0 0))
   )
+  (wire (pts (xy 54.61 94.615) (xy 54.61 90.17))
+    (stroke (width 0) (type default) (color 0 0 0 0))
+  )
   (wire (pts (xy 116.205 121.92) (xy 96.52 121.92))
     (stroke (width 0) (type default) (color 0 0 0 0))
@@
     (stroke (width 0) (type default) (color 0 0 0 0))
   )
+  (wire (pts (xy 116.205 94.615) (xy 54.61 94.615))
+    (stroke (width 0) (type default) (color 0 0 0 0))
+  )
   (wire (pts (xy 106.68 107.315) (xy 106.68 119.38))
     (stroke (width 0) (type default) (color 0 0 0 0))
@@
     (stroke (width 0) (type default) (color 0 0 0 0))
   )
-  (wire (pts (xy 106.68 82.55) (xy 106.68 107.315))
+  (wire (pts (xy 106.68 82.55) (xy 106.68 98.425))
     (stroke (width 0) (type default) (color 0 0 0 0))
   )
@@
     (stroke (width 0) (type default) (color 0 0 0 0))
   )
+  (wire (pts (xy 77.47 98.425) (xy 106.68 98.425))
+    (stroke (width 0) (type default) (color 0 0 0 0))
+  )
+  (wire (pts (xy 62.23 98.425) (xy 69.85 98.425))
+    (stroke (width 0) (type default) (color 0 0 0 0))
+  )
+  (wire (pts (xy 62.23 90.17) (xy 69.85 90.17))
+    (stroke (width 0) (type default) (color 0 0 0 0))
+  )
   (wire (pts (xy 111.125 77.47) (xy 111.125 102.235))
     (stroke (width 0) (type default) (color 0 0 0 0))
@@
     (stroke (width 0) (type default) (color 0 0 0 0))
   )
+  (wire (pts (xy 106.68 98.425) (xy 106.68 107.315))
+    (stroke (width 0) (type default) (color 0 0 0 0))
+  )
   (wire (pts (xy 116.205 94.615) (xy 116.205 121.92))
     (stroke (width 0) (type default) (color 0 0 0 0))
   )
-  (wire (pts (xy 102.87 85.09) (xy 102.87 104.775))
+  (wire (pts (xy 102.87 90.17) (xy 102.87 104.775))
+    (stroke (width 0) (type default) (color 0 0 0 0))
+  )
+  (wire (pts (xy 102.87 85.09) (xy 102.87 90.17))
     (stroke (width 0) (type default) (color 0 0 0 0))
   )
@@
     (stroke (width 0) (type default) (color 0 0 0 0))
   )
+  (wire (pts (xy 77.47 90.17) (xy 102.87 90.17))
+    (stroke (width 0) (type default) (color 0 0 0 0))
+  )
   (wire (pts (xy 116.205 81.915) (xy 116.205 94.615))
     (stroke (width 0) (type default) (color 0 0 0 0))
@@
     (stroke (width 0) (type default) (color 0 0 0 0))
   )
+  (wire (pts (xy 54.61 94.615) (xy 54.61 98.425))
+    (stroke (width 0) (type default) (color 0 0 0 0))
+  )
   (wire (pts (xy 102.87 104.775) (xy 102.87 116.84))
     (stroke (width 0) (type default) (color 0 0 0 0))
@@
   (wire (pts (xy 116.205 94.615) (xy 122.555 94.615))
     (stroke (width 0) (type default) (color 0 0 0 0))
+  )
+  (symbol (lib_id "Connector_Generic:Conn_01x01") (at 49.53 94.615 180) (unit 1)
+    (in_bom yes) (on_board yes)
+    (property "Reference" "J6" (id 0) (at 50.165 92.075 0)
+      (effects (font (size 1.27 1.27)) (justify left))
+    )
+    (property "Value" "3V3" (id 1) (at 46.355 94.615 0)
+      (effects (font (size 1.27 1.27)) (justify left))
+    )
+    (property "Footprint" "user:PinHole_1x01" (id 2) (at 49.53 94.615 0)
+      (effects (font (size 1.27 1.27)) hide)
+    )
+    (property "Datasheet" "~" (id 3) (at 49.53 94.615 0)
+      (effects (font (size 1.27 1.27)) hide)
+    )
+    (pin "1")
   )
   (symbol (lib_id "power:GND") (at 107.95 77.47 180) (unit 1)
@@
     )
     (pin "1")
+  )
+  (symbol (lib_id "Device:R") (at 73.66 90.17 90) (unit 1)
+    (in_bom yes) (on_board yes)
+    (property "Reference" "R1" (id 0) (at 73.66 87.63 90))
+    (property "Value" "R" (id 1) (at 73.66 90.17 90))
+    (property "Footprint" "Resistor_SMD:R_0402_1005Metric" (id 2) (at 73.66 91.948 90)
+      (effects (font (size 1.27 1.27)) hide)
+    )
+    (property "Datasheet" "~" (id 3) (at 73.66 90.17 0)
+      (effects (font (size 1.27 1.27)) hide)
+    )
+    (property "LCSC" "C25900" (id 4) (at 73.66 90.17 0)
+      (effects (font (size 1.27 1.27)) hide)
+    )
+    (pin "1")
+    (pin "2")
   )
   (symbol (lib_id "Switch:SW_Push") (at 112.395 149.225 0) (unit 1)
@@
     (pin "1")
   )
+  (symbol (lib_id "Jumper:SolderJumper_2_Bridged") (at 58.42 90.17 0) (unit 1)
+    (in_bom yes) (on_board yes) (fields_autoplaced)
+    (property "Reference" "JP1" (id 0) (at 58.42 85.3145 0))
+    (property "Value" "SolderJumper_2_Bridged" (id 1) (at 58.42 88.0896 0))
+    (property "Footprint" "Jumper:SolderJumper-2_P1.3mm_Bridged_Pad1.0x1.5mm" (id 2) (at 58.42 90.17 0)
+      (effects (font (size 1.27 1.27)) hide)
+    )
+    (property "Datasheet" "~" (id 3) (at 58.42 90.17 0)
+      (effects (font (size 1.27 1.27)) hide)
+    )
+    (pin "1")
+    (pin "2")
+  )
+  (symbol (lib_id "Device:R") (at 73.66 98.425 90) (unit 1)
+    (in_bom yes) (on_board yes)
+    (property "Reference" "R2" (id 0) (at 73.66 101.6 90))
+    (property "Value" "R" (id 1) (at 73.66 98.425 90))
+    (property "Footprint" "Resistor_SMD:R_0402_1005Metric" (id 2) (at 73.66 100.203 90)
+      (effects (font (size 1.27 1.27)) hide)
+    )
+    (property "Datasheet" "~" (id 3) (at 73.66 98.425 0)
+      (effects (font (size 1.27 1.27)) hide)
+    )
+    (property "LCSC" "C25900" (id 4) (at 73.66 98.425 0)
+      (effects (font (size 1.27 1.27)) hide)
+    )
+    (pin "1")
+    (pin "2")
+  )
+  (symbol (lib_id "Jumper:SolderJumper_2_Bridged") (at 58.42 98.425 0) (unit 1)
+    (in_bom yes) (on_board yes)
+    (property "Reference" "JP2" (id 0) (at 58.42 102.235 0))
+    (property "Value" "SolderJumper_2_Bridged" (id 1) (at 59.69 104.14 0))
+    (property "Footprint" "Jumper:SolderJumper-2_P1.3mm_Bridged_Pad1.0x1.5mm" (id 2) (at 58.42 98.425 0)
+      (effects (font (size 1.27 1.27)) hide)
+    )
+    (property "Datasheet" "~" (id 3) (at 58.42 98.425 0)
+      (effects (font (size 1.27 1.27)) hide)
+    )
+    (pin "1")
+    (pin "2")
+  )
   (symbol (lib_id "power:GND") (at 104.14 146.05 270) (unit 1)
     (in_bom yes) (on_board yes)
@@
       (reference "J5") (unit 1) (value "3V3_EN") (footprint "user:PinHole_1x01")
     )
+    (path "/173fcdac-c021-4747-b471-a941df484443"
+      (reference "J6") (unit 1) (value "3V3") (footprint "user:PinHole_1x01")
+    )
+    (path "/68253e88-4faf-40f2-b038-54be1d22b44f"
+      (reference "JP1") (unit 1) (value "SolderJumper_2_Bridged") (footprint "Jumper:SolderJumper-2_P1.3mm_Bridged_Pad1.0x1.5mm")
+    )
+    (path "/7786c7dc-6b6b-460a-9c03-ecd7747b78ad"
+      (reference "JP2") (unit 1) (value "SolderJumper_2_Bridged") (footprint "Jumper:SolderJumper-2_P1.3mm_Bridged_Pad1.0x1.5mm")
+    )
+    (path "/25b39db8-8576-4473-b331-b912323e85f4"
+      (reference "R1") (unit 1) (value "R") (footprint "Resistor_SMD:R_0402_1005Metric")
+    )
+    (path "/6b5f3da8-29f9-42ad-aa8f-ad2b128165de"
+      (reference "R2") (unit 1) (value "R") (footprint "Resistor_SMD:R_0402_1005Metric")
+    )
     (path "/fb49aa4f-1335-4636-a802-241b030c2abc"
